File: schematics/kikad/arduino-midi-cv.kicad_pcb (KiCad board)
At the start: 2 copper layers, 64 parts, among them J1 Velocity, J2 GATE OUT, J3 Bend Out, J4 MOD WHEEL, J5 V/oct OUT, Q1 BC548, Q2 BC548, U1 TL074, U2 6N137

Commit message: There has been some work done, a long time a go I have no idea what
Parts:
- removed LED_Bend+1: Green LED, LED_THT:LED_D5.0mm
- removed LED_Bend-1: Red LED, LED_THT:LED_D5.0mm
- removed R4, R5: 10R, Resistor_THT:R_Axial_DIN0207_L6.3mm_D2.5mm_P10.16mm_Horizontal
- added ?: , , F.Cu at (170.8, 70.5)
- added ?: , , F.Cu at (156.6, 139.3)
- added ?: , , F.Cu at (127.9, 70.6)
- added C11: 100nF, Capacitor_THT:C_Disc_D3.0mm_W1.6mm_P2.50mm, B.Cu at (139.3, 118.9)
- added C12: 100nF, Capacitor_THT:C_Disc_D3.0mm_W1.6mm_P2.50mm, B.Cu at (139.4, 114.0)
- added FB1: FerriteBead, Resistor_THT:R_Axial_DIN0207_L6.3mm_D2.5mm_P10.16mm_Horizontal, F.Cu at (152.4, 125.7)
- added FB2: FerriteBead, Resistor_THT:R_Axial_DIN0207_L6.3mm_D2.5mm_P10.16mm_Horizontal, F.Cu at (152.3, 138.3)
- added J6: Power connector, Connector_JST:JST_XH_B5B-XH-A_1x05_P2.50mm_Vertical, F.Cu at (159.3, 123.3)
- added J7: Eurorack power connector, Connector_IDC:IDC-Header_2x08_P2.54mm_Vertical, F.Cu at (168.9, 133.3)
- added LED_Bend1: LED_RG, LED_THT:LED_D5.0mm, B.Cu at (158.9, 172.5)
- added R32: 0, Resistor_SMD:R_0805_2012Metric_Pad1.20x1.40mm_HandSolder, B.Cu at (130.8, 80.0)
- added R33: 1k, Resistor_THT:R_Axial_DIN0207_L6.3mm_D2.5mm_P10.16mm_Horizontal, F.Cu at (147.7, 88.1)
- added SW1: RotaryEncoder_Switch, Rotary_Encoder:RotaryEncoder_Alps_EC11E-Switch_Vertical_H20mm, B.Cu at (142.2, 118.8)
- added U3: OLED_Display_SPI, Dr_McFishs_misc_footprints:SPI Oled dislay SH1106, B.Cu at (156.8, 69.5)
- A1: moved to F.Cu
- C3, C4: value 10uF -> 22uF
- D1: footprint Diode_THT:D_DO-35_SOD27_P7.62mm_Horizontal -> Diode_THT:D_DO-35_SOD27_P2.54mm_Vertical_AnodeUp
- D2, D3: footprint Diode_THT:D_DO-41_SOD81_P2.54mm_Vertical_AnodeUp -> Diode_THT:D_DO-41_SOD81_P12.70mm_Horizontal
- D4, LED_MOD1, LED_V/oct1, LED_VELOCITY1: moved to B.Cu
- J1, J2, J3, J4, J5: footprint Connector_PinHeader_1.00mm:PinHeader_1x02_P1.00mm_Vertical -> Library:Jack breakcout cables
- J_MIDI_OUT1, J_MIDI_THRU1: footprint Connector_PinHeader_1.00mm:PinHeader_1x05_P1.00mm_Vertical -> Library:SIP-2
- Q1, Q2: footprint Package_TO_SOT_THT:TO-92L_Inline_Wide -> Package_TO_SOT_THT:TO-92_Inline
- R12: footprint Resistor_THT:R_Axial_DIN0207_L6.3mm_D2.5mm_P10.16mm_Horizontal -> Resistor_THT:R_Axial_DIN0207_L6.3mm_D2.5mm_P2.54mm_Vertical
- R13: footprint Resistor_THT:R_Axial_DIN0207_L6.3mm_D2.5mm_P10.16mm_Horizontal -> Resistor_THT:R_Axial_DIN0207_L6.3mm_D2.5mm_P7.62mm_Horizontal
- R25: value 10k -> 100k; footprint Resistor_THT:R_Axial_DIN0207_L6.3mm_D2.5mm_P10.16mm_Horizontal -> Resistor_THT:R_Axial_DIN0207_L6.3mm_D2.5mm_P2.54mm_Vertical
- R27: value 10k -> 100k
- R3: value 10k -> 1k
- RV1: footprint Potentiometer_THT:Potentiometer_ACP_CA9-V10_Vertical -> Potentiometer_THT:Potentiometer_Bourns_3296W_Vertical
- moved J_MIDI_OUT1 160.6 mm to (127.9, 115.1), turned to -90 degrees
- moved J1 148.4 mm to (172.2, 158.5), turned to 90 degrees
- moved C5 148.2 mm to (129.9, 98.0), turned to -90 degrees
- moved C6 141.3 mm to (155.8, 158.1)
- moved C10 138.0 mm to (139.7, 149.5)
- moved U2 138.0 mm to (127.9, 110.9), turned to 90 degrees
- moved J4 137.8 mm to (128.3, 156.2), turned to 90 degrees
- moved R19 135.0 mm to (126.9, 150.0)
- moved D6 132.5 mm to (140.1, 84.7)
- moved R28 129.5 mm to (136.8, 161.4), turned to 180 degrees
- moved J5 129.4 mm to (126.5, 144.9), turned to -90 degrees
- moved R21 126.4 mm to (131.8, 146.4)
- moved R18 125.6 mm to (127.0, 165.1), turned to -90 degrees
- moved R14 122.1 mm to (167.1, 141.0), turned to -90 degrees
- moved R8 121.5 mm to (140.0, 164.6), turned to 180 degrees
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Connections:
- net Net-(A1-Pad12) renamed V/oct PWM
- net Net-(A1-Pad13) renamed Pitch Wheel PWM
- net Net-(R13-Pad1) renamed MIDI RX
- A1 pad 1: unconnected-(A1-Pad1) -> SPI Reset
- A1 pad 10: unconnected-(A1-Pad10) -> SPI DC
- A1 pad 11: unconnected-(A1-Pad11) -> SPI CS
- A1 pad 14: Net-(R8-Pad1) -> SPI MOSI
- A1 pad 15: Net-(R6-Pad1) -> unconnected-(A1-Pad15)
- A1 pad 16: unconnected-(A1-Pad16) -> SPI SLK
- A1 pad 22: unconnected-(A1-Pad22) -> Encoder Button
- A1 pad 30: +12V -> Net-(A1-Pad30)
- A1 pad 5: unconnected-(A1-Pad5) -> Encoder CLK
- A1 pad 6: Net-(A1-Pad6) -> Encoder DT
- A1 pad 7: unconnected-(A1-Pad7) -> Gate Pin
- A1 pad 8: unconnected-(A1-Pad8) -> Velocity PWM
- A1 pad 9: unconnected-(A1-Pad9) -> Mod Wheel PWM
- C8 pad 1: Net-(R8-Pad2) -> Net-(C8-Pad1)
- D5 pad 2: Net-(R6-Pad1) -> Net-(D5-Pad2)
- D6 pad 1: Net-(R6-Pad1) -> Net-(D5-Pad2)
- R10 pad 1: Net-(A1-Pad6) -> Velocity PWM
- R14 pad 1: Net-(A1-Pad6) -> Velocity PWM
- R18 pad 1: Net-(R6-Pad1) -> Gate Pin
- R22 pad 2: Net-(R8-Pad2) -> Mod Wheel PWM
- R30 pad 2: Net-(J5-PadT) -> V/oct  Out
- R6 pad 1: Net-(R6-Pad1) -> Net-(D5-Pad2)
- R6 pad 2: Net-(J2-PadT) -> Gate  Out
- R8 pad 1: Net-(R8-Pad1) -> Mod Wheel PWM
- R8 pad 2: Net-(R8-Pad2) -> Net-(C8-Pad1)
- U1 pad 12: Net-(R8-Pad2) -> Net-(C8-Pad1)
Routing:
- net V/oct PWM: track 0.00 -> 107.1 mm, vias 0 -> 2
- net Velocity PWM: track 0.00 -> 103.6 mm
- net Gate Pin: track 0.00 -> 91.1 mm
- net Mod Wheel PWM: track 0.00 -> 90.4 mm
- net Gate  Out: track 0.00 -> 58.9 mm
- net V/oct  Out: track 0.00 -> 55.4 mm, vias 0 -> 1
- net Pitch Wheel PWM: track 0.00 -> 51.2 mm
- net Encoder Button: track 0.00 -> 42.6 mm
- net +12V: track 142.2 -> 101.7 mm, vias 2 -> 0
- net SPI Reset: track 0.00 -> 40.0 mm
- net Earth: track 157.5 -> 121.3 mm, vias 2 -> 30
- net unconnected-(A1-Pad28): track 35.6 -> 0.00 mm
- net unconnected-(A1-Pad26): track 35.6 -> 0.00 mm
- net unconnected-(A1-Pad25): track 35.6 -> 0.00 mm
- net unconnected-(A1-Pad24): track 35.6 -> 0.00 mm
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- added copper zone on B.Cu, net Earth
- added copper zone on F.Cu, net Earth
Other:
- board outline added: 49.5 x 109.2 mm
